File: cc1101/mcu.kicad_sch (KiCad schematic)
At the start: 22 parts, among them J104 Conn_ARM_JTAG_SWD_10, J402 Conn_01x02, SW101 Alps SKRTLAE010, U102 STM32F401RCT6, Y101 8MHz 20pF

Commit message: cc1quack: Add specialized switch footprint
Specialize the ALPS SKRTLAE010 to include project-specific 3D model
paths.

Signed-off-by: Andreas Sandberg <andreas@sandberg.uk>
Parts:
- SW101: footprint Button_Switch_SMD:SW_Push_1P1T-MP_NO_Horizontal_Alps_SKRTLAE010 -> quack:SW_Push_1P1T-MP_NO_Horizontal_Alps_SKRTLAE010
Changed lines of the file:
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@@
       (effects (font (size 1.27 1.27)) (justify right))
     )
-    (property "Footprint" "Button_Switch_SMD:SW_Push_1P1T-MP_NO_Horizontal_Alps_SKRTLAE010" (at 77.47 140.97 0)
+    (property "Footprint" "quack:SW_Push_1P1T-MP_NO_Horizontal_Alps_SKRTLAE010" (at 77.47 140.97 0)
       (effects (font (size 1.27 1.27)) hide)
     )
