File: cc1101/cc1quack.kicad_sch (KiCad schematic)
At the start: 28 parts, among them J103 Conn_01x06_Pin

Commit message: cc1quack: Specialize LiteOn LTST C19HE1WT footprint
Specialize LiteOn LTST C19HE1WT footprint to include 3D models.

Signed-off-by: Andreas Sandberg <andreas@sandberg.uk>
Parts:
- D103, D104, D105: footprint LED_SMD:LED_LiteOn_LTST-C19HE1WT -> quack:LED_LiteOn_LTST-C19HE1WT
Changed lines of the file:
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@@
       (effects (font (size 1.27 1.27)) (justify right))
     )
-    (property "Footprint" "LED_SMD:LED_LiteOn_LTST-C19HE1WT" (at 222.25 36.83 0)
+    (property "Footprint" "quack:LED_LiteOn_LTST-C19HE1WT" (at 222.25 36.83 0)
       (effects (font (size 1.27 1.27)) hide)
     )
@@
       (effects (font (size 1.27 1.27)) (justify right))
     )
-    (property "Footprint" "LED_SMD:LED_LiteOn_LTST-C19HE1WT" (at 260.35 36.83 0)
+    (property "Footprint" "quack:LED_LiteOn_LTST-C19HE1WT" (at 260.35 36.83 0)
       (effects (font (size 1.27 1.27)) hide)
     )
@@
       (effects (font (size 1.27 1.27)) (justify right))
     )
-    (property "Footprint" "LED_SMD:LED_LiteOn_LTST-C19HE1WT" (at 180.34 36.83 0)
-      (effects (font (size 1.27 1.27)) hide)
-    )
+    (property "Footprint" "quack:LED_LiteOn_LTST-C19HE1WT" (at 180.34 36.83 0)
+      (effects (font (size 1.27 1.27)) hide)
+    )
